Commit message: Update src folder
Added some dynamic arguments to easily change between simulation topics and real robot ones

File: src/husky/husky_description/urdf/husky.urdf.xacro (robot description, xacro)
@@ -25,5 +25,5 @@
   <xacro:arg name="laser_xyz" default="$(optenv HUSKY_LMS1XX_XYZ 0.2206 0.0 0.00635)" />
   <xacro:arg name="laser_rpy" default="$(optenv HUSKY_LMS1XX_RPY 0.0 0.0 0.0)" />
-  <xacro:arg name="kinect_enabled" default="true" />
+  <xacro:arg name="kinect_enabled" default="false" />
   <xacro:arg name="kinect_xyz" default="$(optenv HUSKY_KINECT_XYZ 0 0 0)" />
   <xacro:arg name="kinect_rpy" default="$(optenv HUSKY_KINECT_RPY 0 0.18 3.14)" />
@@ -80,6 +80,5 @@
     <inertial>
       <mass value="46.034" />
-      <!--origin xyz="-0.00065 -0.085 0.062" /-->
-      <origin xyz="0.0 0.0 0.062" rpy="0 0 0" />
+      <origin xyz="-0.00065 -0.085 0.062" />
       <inertia ixx="0.6022" ixy="-0.02364" ixz="-0.1197" iyy="1.7386" iyz="-0.001544" izz="2.0296" />
     </inertial>
